File: KiCAD Files/ACS712-module.kicad_sch (KiCad schematic)
At the start: 23 parts, among them J1 Banana plug, J2 Banana plug, J3 power, J4 USB_B_Mini, U1 ACS712

Commit message: update
Other:
- note added: "Mounting holes"
- note added: "Power LED"
- note added: "Power flags"
- note added: "Sensor"
- note added: "USB power connector"
Changed lines of the file:
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@@
     (stroke (width 0) (type default))
+  )
+  (text "USB power connector" (at 45.72 70.485 0)
+    (effects (font (size 1.27 1.27)) (justify left bottom))
+  )
+  (text "Power flags" (at 132.715 168.91 0)
+    (effects (font (size 1.27 1.27)) (justify left bottom))
+  )
+  (text "Power LED" (at 91.44 77.47 0)
+    (effects (font (size 1.27 1.27)) (justify left bottom))
+  )
+  (text "Mounting holes" (at 94.615 154.94 0)
+    (effects (font (size 1.27 1.27)) (justify left bottom))
+  )
+  (text "Sensor" (at 165.1 69.85 0)
+    (effects (font (size 1.27 1.27)) (justify left bottom))
   )
   (label "Vout" (at 175.26 95.25 0) (fields_autoplaced)
