File: KiCAD Files/ACS712-module.kicad_sch (KiCad schematic)
At the start: 23 parts, among them J1 Banana plug, J2 Banana plug, J3 power, J4 USB_B_Mini, U1 ACS712

Commit message: update
Parts:
- removed J3: power, Connector_PinHeader_2.54mm:PinHeader_1x02_P2.54mm_Vertical, symbol Connector:Conn_01x02_Pin
- removed J4: USB_B_Mini, Connector_USB:USB_Mini-B_Lumberg_2486_01_Horizontal, symbol Connector:USB_B_Mini
- removed JP4: Jumper_3_Open, Connector_PinHeader_2.54mm:PinHeader_1x03_P2.54mm_Vertical, symbol Jumper:Jumper_3_Open
- added C5, C6: 10uF, Capacitor_SMD:C_0805_2012Metric, symbol Device:C_Small
- added J5: Barrel_Jack_MountingPin, Connector_BarrelJack:BarrelJack_Wuerth_6941xx301002, symbol Connector:Barrel_Jack_MountingPin
- added U2: AMS1117-5.0, Package_TO_SOT_SMD:SOT-223-3_TabPin2, symbol Regulator_Linear:AMS1117-5.0
- R1: value 680R -> 1k3
Connections:
- net +5V: now also C6.1, U2.2 (VO); no longer R1.1
- net GND: now also D1.1 (K), C5.2, C6.2, J5.2, U2.1 (GND); no longer D1.2 (A)
- net at R1.2: now also D1.2 (A); no longer D1.1 (K)
- new net +12V: C5.1, J5.1, R1.1, U2.3 (VI)
- no-connect marks 8 -> 5
Other:
- note added: "Barrel jack 12V power connector"
- note added: "TO-DO: - Povećati fontove jer su nečitljivi - barrel jack 3d model"
- note removed: "Power LED"
- note removed: "USB power connector"
- moved on the sheet: D1, R1

Commit message: update
Other:
- note removed: "TO-DO: - Povećati fontove jer su nečitljivi - barrel jack 3d model"
- moved on the sheet: C1, C2, C3, C4, C5, C6, D1, H1, H2, H3, H4, J1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
