File: KiCAD Files/ACS712-module.kicad_pcb (KiCad board)
At the start: 2 copper layers, 70 x 55 mm, 24 parts, among them J1 Banana plug, J2 Banana plug, J3 power, J4 USB_B_Mini, U1 ACS712

Commit message: update
Parts:
- removed G***: LOGO, Library:tvz
- removed J3: power, Connector_PinHeader_2.54mm:PinHeader_1x02_P2.54mm_Vertical
- removed J4: USB_B_Mini, Connector_USB:USB_Mini-B_Lumberg_2486_01_Horizontal
- removed JP4: Jumper_3_Open, Connector_PinHeader_2.54mm:PinHeader_1x03_P2.54mm_Vertical
- added C5: 10uF, Capacitor_SMD:C_0805_2012Metric, F.Cu at (158.5, 113.5)
- added C6: 10uF, Capacitor_SMD:C_0805_2012Metric, F.Cu at (158.5, 98.5)
- added J5: Barrel_Jack_MountingPin, Connector_BarrelJack:BarrelJack_Wuerth_6941xx301002, F.Cu at (165.5, 105.1)
- added U2: AMS1117-5.0, Package_TO_SOT_SMD:SOT-223-3_TabPin2, F.Cu at (158.5, 105.5)
- R1: value 680R -> 1k3
- moved R1 19.7 mm to (172.2, 115.8)
- moved D1 19.3 mm to (172.3, 113.0), turned to 0 degrees
Connections:
- D1 pad 1: Net-(D1-K) -> GND
- D1 pad 2: GND -> Net-(D1-A)
- R1 pad 1: +5V -> +12V
- R1 pad 2: Net-(D1-K) -> Net-(D1-A)
Routing:
- net +12V: track 0.00 -> 29.3 mm
- net Net-(J3-Pin_1): track 14.0 -> 0.00 mm
- net Net-(D1-K): track 5.26 -> 0.00 mm
- net Net-(D1-A): track 0.00 -> 4.96 mm
- net +5V: track 49.9 -> 52.5 mm
- net /Vout: track 41.4 -> 39.8 mm
- removed copper zone on F.Cu, net Net-(J4-VBUS)
Other:
- board text added: "ACS712/723"
- board text added: "TVZ ACS712/723 v1rev1"
- board text removed: "5V"
- board text removed: "ACS712"
- board text removed: "TVZ ACS712 Current sensing module v1rev1"

Commit message: update
Parts:
- added G***: LOGO, Library:tvz2, F.Cu at (114.8, 93.0)

Commit message: update
Parts:
- moved JP1 0.16 mm to (119.3, 105.8)
- moved JP3 0.16 mm to (139.7, 105.8)
Changed lines of the file:
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@@
 	(footprint "Connector_PinHeader_2.54mm:PinHeader_1x02_P2.54mm_Vertical"
 		(layer "F.Cu")
-		(at 119.5 105.775 180)
+		(at 119.34 105.775 180)
 		(descr "Through hole straight pin header, 1x02, 2.54mm pitch, single row")
 		(tags "Through hole pin header THT 1x02 2.54mm single row")
@@
 	(footprint "Connector_PinHeader_2.54mm:PinHeader_1x02_P2.54mm_Vertical"
 		(layer "F.Cu")
-		(at 139.5 105.775 180)
+		(at 139.66 105.775 180)
 		(descr "Through hole straight pin header, 1x02, 2.54mm pitch, single row")
 		(tags "Through hole pin header THT 1x02 2.54mm single row")
@@
 	)
 	(segment
-		(start 124.5 105.45)
-		(end 124.5 107.5)
+		(start 119.75 108)
+		(end 119.34 107.59)
 		(width 0.6)
 		(layer "F.Cu")
@@
 	)
 	(segment
-		(start 124 108)
+		(start 124.5 105.45)
 		(end 124.5 107.5)
 		(width 0.6)
@@
 	)
 	(segment
-		(start 119.5 105.775)
-		(end 119.5 107.5)
+		(start 124 108)
+		(end 124.5 107.5)
 		(width 0.6)
 		(layer "F.Cu")
@@
 	)
 	(segment
-		(start 120 108)
-		(end 124 108)
+		(start 124 108)
+		(end 119.75 108)
 		(width 0.6)
 		(layer "F.Cu")
@@
 	)
 	(segment
-		(start 119.5 107.5)
-		(end 120 108)
+		(start 119.34 107.59)
+		(end 119.34 105.775)
 		(width 0.6)
 		(layer "F.Cu")
@@
 	)
 	(segment
-		(start 139.5 105.775)
-		(end 139.5 107.5)
+		(start 144 108)
+		(end 140.25 108)
 		(width 0.6)
 		(layer "F.Cu")
@@
 	)
 	(segment
-		(start 139.5 107.5)
-		(end 140 108)
+		(start 144 108)
+		(end 144.46 107.54)
 		(width 0.6)
 		(layer "F.Cu")
@@
 	)
 	(segment
-		(start 144 108)
-		(end 144.46 107.54)
+		(start 139.66 107.41)
+		(end 139.66 105.775)
 		(width 0.6)
 		(layer "F.Cu")
@@
 	)
 	(segment
-		(start 140 108)
-		(end 144 108)
+		(start 140.25 108)
+		(end 139.66 107.41)
 		(width 0.6)
 		(layer "F.Cu")

Commit message: update
Routing:
- net GND: vias 5 -> 12
